File: board/motion-led.kicad_pcb (KiCad board)
At the start: 2 copper layers, 63.5 x 36.8 mm, 10 parts, among them J0 Barrel_Jack, J1 AM312, J2 LED PINs, Q0 2N7002, Q1 2N7002, Q2 2N7002, U0 WeMos_D1_mini

Commit message: Finalize PCB
Parts:
- moved J1 43.2 mm to (99.6, 97.3), turned to 0 degrees
- moved U0 2.97 mm to (104.6, 97.3)
Routing:
- net GND: track 60.1 -> 10.7 mm, vias 0 -> 3
- net Net-(J1-Pad2): track 40.3 -> 5.08 mm
- net Net-(J1-Pad3): track 31.4 -> 16.4 mm
- net Net-(R0-Pad2): track 8.17 -> 5.16 mm
- net Net-(R1-Pad2): track 7.98 -> 5.05 mm
- net Net-(R2-Pad2): track 8.51 -> 5.58 mm
- net Net-(J0-Pad1): track 27.9 -> 26.2 mm
- added copper zone on B.Cu, net GND
Other:
- board size 63.5 x 36.8 mm -> 62.7 x 36.8 mm
